File: rigel-a-rx/rigel-a-hw/rigel-a-hw.kicad_pcb (KiCad board)
At the start: 2 copper layers, 0 parts

Commit message: Pretty much finish layout
Parts:
- added C1: 0.47uF, Capacitor_SMD:C_0603_1608Metric, B.Cu at (126.3, 110.9)
- added C10: 100nF, Capacitor_SMD:C_0402_1005Metric, B.Cu at (117.4, 108.3)
- added C11: 100nF, Capacitor_SMD:C_0402_1005Metric, B.Cu at (126.1, 106.1)
- added C12: 100nF, Capacitor_SMD:C_0402_1005Metric, B.Cu at (120.9, 104.6)
- added C13: 100nF, Capacitor_SMD:C_0402_1005Metric, B.Cu at (114.3, 108.8)
- added C14: 1uF, Capacitor_SMD:C_0603_1608Metric, B.Cu at (126.7, 101.6)
- added C15: 1uF, Capacitor_SMD:C_0603_1608Metric, B.Cu at (132.9, 102.4)
- added C16: 4.7uF, Capacitor_SMD:C_0603_1608Metric, B.Cu at (125.7, 104.7)
- added C17: 10nF, Capacitor_SMD:C_0402_1005Metric, B.Cu at (115.9, 113.8)
- added C18: 10pF, Capacitor_SMD:C_0402_1005Metric, B.Cu at (116.8, 112.5)
- added C19: 100nF, Capacitor_SMD:C_0402_1005Metric, B.Cu at (126.1, 107.3)
- added C2: 33pF, Capacitor_SMD:C_0402_1005Metric, B.Cu at (119.9, 114.5)
- added C3: 100nF, Capacitor_SMD:C_0402_1005Metric, B.Cu at (123.5, 109.4)
- added C4: 100nF, Capacitor_SMD:C_0402_1005Metric, B.Cu at (117.7, 114.5)
- added C5: 100nF, Capacitor_SMD:C_0402_1005Metric, B.Cu at (123.5, 110.6)
- added C6: 100nF, Capacitor_SMD:C_0402_1005Metric, B.Cu at (123.5, 111.8)
- added C7: 100nF, Capacitor_SMD:C_0402_1005Metric, B.Cu at (118.8, 114.5)
- added C8: 100nF, Capacitor_SMD:C_0402_1005Metric, B.Cu at (126.8, 109.2)
- added C9: 4.7uF, Capacitor_SMD:C_0603_1608Metric, B.Cu at (112.3, 103.0)
- added IC1: BALFHB-WL-02D3, jlc:BALFHBWL02D3, F.Cu at (111.9, 111.1)
- added J1: Conn_01x03_Pin, Connector_PinSocket_2.54mm:PinSocket_1x03_P2.54mm_Vertical, B.Cu at (128.4, 118.3)
- added J3: Conn_01x03_Pin, Connector_PinSocket_2.54mm:PinSocket_1x03_P2.54mm_Vertical, B.Cu at (116.4, 101.8)
- added L1: GZ2012D601TF, jlc:L0805, B.Cu at (124.3, 102.1)
- added LED1: 0805G_(Green), jlc:LED0805-R-RD, B.Cu at (104.8, 103.6)
- added LED2: 0805G_(Green), jlc:LED0805-R-RD, B.Cu at (107.4, 103.6)
- added R1: 5.1k, Resistor_SMD:R_0402_1005Metric, B.Cu at (127.0, 114.8)
- added R2: 5.1k, Resistor_SMD:R_0402_1005Metric, B.Cu at (125.0, 114.8)
- added R3: 4.7k, Resistor_SMD:R_0402_1005Metric, B.Cu at (115.3, 110.5)
- added R4: 220, Resistor_SMD:R_0402_1005Metric, B.Cu at (114.2, 113.0)
- added R5: 68, Resistor_SMD:R_0603_1608Metric, B.Cu at (110.0, 105.4)
- added R6: 68, Resistor_SMD:R_0603_1608Metric, B.Cu at (110.9, 101.1)
- added U1: STM32WLE5C8Ux, Package_DFN_QFN:QFN-48-1EP_7x7mm_P0.5mm_EP5.6x5.6mm, F.Cu at (120.6, 109.1)
- added U2: XC6206P332MR, jlc:SOT-23-3_L2.9-W1.6-P1.90-LS2.8-BR, B.Cu at (129.9, 102.3)
- added U3: CH340X, jlc:MSOP-10_L3.0-W3.0-P0.50-LS5.0-BL, B.Cu at (114.8, 106.3)
- added U4: TYPE-C_16PIN_2MD(073), jlc:USB-C-SMD_TYPE-C-6PIN-2MD-073, B.Cu at (131.1, 109.7)
- added U5: X1G004131004200, jlc:OSC-SMD_4P-L2.0-W1.6-BL_EPSON_TG-5006CJ-19H, B.Cu at (115.5, 115.7)
- added U6: KH-SMA-K513-G, jlc:ANT-TH_KH-SMA-K513-G, B.Cu at (104.6, 109.8)
Routing:
- net USBD-: track 0.00 -> 40.4 mm
- net +3.3V: track 0.00 -> 38.9 mm, vias 0 -> 11
- net USBD+: track 0.00 -> 36.4 mm
- net +5V: track 0.00 -> 17.1 mm, vias 0 -> 2
- net +1V5: track 0.00 -> 12.7 mm, vias 0 -> 2
- net /JTCK/SWCLK: track 0.00 -> 10.5 mm
- net /TIM1_CH1_LED_1: track 0.00 -> 9.88 mm, vias 0 -> 1
- net Net-(U1-VDDA): track 0.00 -> 8.71 mm, vias 0 -> 1
- net /TIM1_CH2_LED_2: track 0.00 -> 8.09 mm, vias 0 -> 1
- net /BOOT0: track 0.00 -> 8.02 mm, vias 0 -> 1
- net Net-(U4-CC1): track 0.00 -> 7.85 mm, vias 0 -> 2
- net /RESET: track 0.00 -> 7.16 mm, vias 0 -> 1
- net /PB0-VDD_TCXO: track 0.00 -> 7.13 mm, vias 0 -> 1
- net Net-(LED1-A): track 0.00 -> 7.02 mm
- net Net-(IC1-RFI_IN): track 0.00 -> 6.62 mm
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- added copper zone on In2.Cu, net +3.3V
- added copper zone on B.Cu, net GND
- added copper zone on F.Cu, net GND
- added copper zone on In1.Cu, net GND
Other:
- board outline added: 35 x 20 mm
- copper layers 2 -> 4
- board text added: "GND SWCLK SWDIO"
- board text added: "STAT INFO"
- board text added: "SWD"
- board text added: "TX RX GND"
- board text added: "{ "ViaStitching": "0.2", "stitch_zone_0": { "HSpacing": "1.16", "VSpacing": "1.16", "Clearance": "2", "Randomize": false } }"
